File: Hardware/Sparkfun_RS232.brd (EAGLE design)
At the start: 22.9 x 30.5 mm, 16 parts, among them U2 XN04312

Commit message: qc CL items fixed.
Parts:
- C4: device SparkFun:EIA3216 -> SparkFun-Capacitors:EIA3216
- D1: device SparkFun:SOD-323 -> SparkFun-DiscreteSemi:SOD-323
- D4, D5: device SparkFun:LED-1206 -> SparkFun-LED:LED-1206
- U2: device SparkFun:SOT23-6 -> SparkFun-DiscreteSemi:SOT23-6
Connections:
- net N$4: now also D1.A; no longer D1.2
- net RS-IN: now also D1.C; no longer D1.1
Routing:
- net N$1: track 2.89 -> 4.71 mm
