File: Hardware/Sparkfun_RS232.sch (EAGLE design)
At the start: 16 parts, among them U2 XN04312

Commit message: qc CL items fixed.
Parts:
- C4: device SparkFun:CAP_POL1206 -> SparkFun-Capacitors:10UF-16V-10%(TANT)
- D1: device SparkFun:DIODESOD -> SparkFun-DiscreteSemi:DIODEBAS16
- D4: device SparkFun:LED1206 -> SparkFun-LED:LED-RED1206
- D5: device SparkFun:LED1206 -> SparkFun-LED:LED-GREENLARGE
- U2: device SparkFun:XN04312SOT -> SparkFun-DiscreteSemi:XN04312SOT
Other:
- moved on the sheet: R1
Changed lines of the file:
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@@
 <layer number="56" name="wert" color="7" fill="1" visible="no" active="no"/>
 <layer number="57" name="tCAD" color="7" fill="1" visible="no" active="no"/>
+<layer number="59" name="tCarbon" color="7" fill="1" visible="no" active="no"/>
+<layer number="60" name="bCarbon" color="7" fill="1" visible="no" active="no"/>
+<layer number="90" name="Modules" color="5" fill="1" visible="yes" active="yes"/>
 <layer number="91" name="Nets" color="2" fill="1" visible="yes" active="yes"/>
 <layer number="92" name="Busses" color="1" fill="1" visible="yes" active="yes"/>
@@
 <layer number="127" name="_tValues" color="7" fill="1" visible="yes" active="yes"/>
 <layer number="128" name="_bValues" color="7" fill="1" visible="yes" active="yes"/>
+<layer number="129" name="Mask" color="7" fill="1" visible="yes" active="yes"/>
 <layer number="131" name="tAdjust" color="7" fill="1" visible="yes" active="yes"/>
 <layer number="132" name="bAdjust" color="7" fill="1" visible="yes" active="yes"/>
@@
 <layer number="223" name="223bmp" color="7" fill="1" visible="yes" active="yes"/>
 <layer number="224" name="224bmp" color="7" fill="1" visible="yes" active="yes"/>
+<layer number="225" name="225bmp" color="7" fill="1" visible="yes" active="yes"/>
+<layer number="226" name="226bmp" color="7" fill="1" visible="yes" active="yes"/>
+<layer number="227" name="227bmp" color="7" fill="1" visible="yes" active="yes"/>
+<layer number="228" name="228bmp" color="7" fill="1" visible="yes" active="yes"/>
+<layer number="229" name="229bmp" color="7" fill="1" visible="yes" active="yes"/>
+<layer number="230" name="230bmp" color="7" fill="1" visible="yes" active="yes"/>
+<layer number="231" name="231bmp" color="7" fill="1" visible="yes" active="yes"/>
 <layer number="248" name="Housing" color="7" fill="1" visible="yes" active="yes"/>
 <layer number="249" name="Edge" color="7" fill="1" visible="yes" active="yes"/>
@@
 <layer number="251" name="SMDround" color="12" fill="11" visible="no" active="no"/>
 <layer number="254" name="cooling" color="7" fill="1" visible="yes" active="yes"/>
+<layer number="255" name="routoute" color="7" fill="1" visible="yes" active="yes"/>
 </layers>
-<schematic>
+<schematic xreflabel="%F%N/%S" xrefpart="/%S.%C%R">
 <attributes>
 </attributes>
@@
 <part name="FRAME1" library="SparkFun-Aesthetics" deviceset="FRAME-LETTER" device=""/>
 <part name="JP1" library="SparkFun-Connectors" deviceset="DB9" device="FEMALE" value="DB9"/>
-<part name="D4" library="SparkFun" deviceset="LED" device="1206" value="Red"/>
-<part name="D5" library="SparkFun" deviceset="LED" device="1206" value="Grn"/>
-<part name="D1" library="SparkFun" deviceset="DIODE" device="SOD" value="BAS16"/>
-<part name="C4" library="SparkFun" deviceset="CAP_POL" device="1206" value="10uF"/>
+<part name="D4" library="SparkFun-LED" deviceset="LED-RED" device="1206" value="Red"/>
+<part name="D5" library="SparkFun-LED" deviceset="LED-GREEN" device="LARGE" value="Grn"/>
+<part name="D1" library="SparkFun-DiscreteSemi" deviceset="DIODE" device="BAS16" value="BAS16"/>
+<part name="C4" library="SparkFun-Capacitors" deviceset="10UF-16V-10%(TANT)" device="" value="10uF"/>
 <part name="R3" library="SparkFun-Resistors" deviceset="330OHM1/10W1%(0603)" device="" value="330"/>
 <part name="R4" library="SparkFun-Resistors" deviceset="330OHM1/10W1%(0603)" device="" value="330"/>
@@
 <part name="E$1" library="SparkFun" deviceset="FIDUCIAL" device="1X2"/>
 <part name="E$2" library="SparkFun" deviceset="FIDUCIAL" device="1X2"/>
-<part name="U2" library="SparkFun" deviceset="XN04312" device="SOT" value="XN04312"/>
+<part name="U2" library="SparkFun-DiscreteSemi" deviceset="XN04312" device="SOT" value="XN04312"/>
 <part name="LOGO2" library="SparkFun-Aesthetics" deviceset="OSHW-LOGO" device="M"/>
 <part name="LOGO1" library="SparkFun-Aesthetics" deviceset="SFE_LOGO_NAME_FLAME" device=".1_INCH" value="SFE_LOGO_NAME_FLAME.1_INCH"/>
@@
 <instance part="GND7" gate="1" x="154.94" y="99.06"/>
 <instance part="GND8" gate="1" x="144.78" y="68.58"/>
-<instance part="R1" gate="G$1" x="154.94" y="134.62" rot="R90"/>
-<instance part="P+5" gate="1" x="144.78" y="144.78"/>
+<instance part="R1" gate="G$1" x="154.94" y="142.24" rot="R90"/>
+<instance part="P+5" gate="1" x="144.78" y="152.4"/>
 <instance part="GND1" gate="1" x="81.28" y="99.06"/>
 <instance part="JP2" gate="G$1" x="210.82" y="109.22" rot="R180"/>
@@
 </segment>
 <segment>
-<wire x1="154.94" y1="139.7" x2="154.94" y2="142.24" width="0.1524" layer="91"/>
-<wire x1="154.94" y1="142.24" x2="144.78" y2="142.24" width="0.1524" layer="91"/>
-<wire x1="144.78" y1="142.24" x2="144.78" y2="144.78" width="0.1524" layer="91"/>
-<wire x1="144.78" y1="142.24" x2="144.78" y2="124.46" width="0.1524" layer="91"/>
-<junction x="144.78" y="142.24"/>
+<wire x1="154.94" y1="147.32" x2="154.94" y2="149.86" width="0.1524" layer="91"/>
+<wire x1="154.94" y1="149.86" x2="144.78" y2="149.86" width="0.1524" layer="91"/>
+<wire x1="144.78" y1="149.86" x2="144.78" y2="152.4" width="0.1524" layer="91"/>
+<wire x1="144.78" y1="149.86" x2="144.78" y2="124.46" width="0.1524" layer="91"/>
+<junction x="144.78" y="149.86"/>
 <pinref part="R1" gate="G$1" pin="2"/>
 <pinref part="P+5" gate="1" pin="VCC"/>
@@
 </segment>
 <segment>
-<wire x1="149.86" y1="124.46" x2="149.86" y2="127" width="0.1524" layer="91"/>
+<wire x1="149.86" y1="124.46" x2="149.86" y2="132.08" width="0.1524" layer="91"/>
+<wire x1="149.86" y1="132.08" x2="157.48" y2="132.08" width="0.1524" layer="91"/>
 <pinref part="U2" gate="G$1" pin="B2"/>
-<label x="149.86" y="127" size="1.27" layer="95" rot="R180" xref="yes"/>
+<label x="157.48" y="132.08" size="1.27" layer="95" xref="yes"/>
 </segment>
 <segment>
@@
 </segment>
 <segment>
-<wire x1="154.94" y1="129.54" x2="154.94" y2="127" width="0.1524" layer="91"/>
+<wire x1="154.94" y1="137.16" x2="154.94" y2="127" width="0.1524" layer="91"/>
 <wire x1="154.94" y1="127" x2="154.94" y2="124.46" width="0.1524" layer="91"/>
 <wire x1="154.94" y1="127" x2="157.48" y2="127" width="0.1524" layer="91"/>
